File: hardware/PiRF/PiRF.kicad_pcb (KiCad board)
At the start: 2 copper layers, 65 x 56 mm, 40 parts, among them J1 CONN_01X02, J2 40HAT, J3 Conn_02x20_Odd_Even, J4 CONN_01X02, J5 Conn_Coaxial, J6 CONN_01X02, U1 CAT24C32, U2 TPS7A19, U3 TS5A23159, U4 TPS2294x, U5 ST_Teseo

Commit message: Order Rev B
Parts:
- removed H1, H2, H5, H7: 3mm_Mounting_Hole, MountingHole:MountingHole_2.1mm
- removed H4, H8: 3mm_Mounting_Hole, project_footprints:NPTH_3mm_ID
- removed TP4, TP6: TestPoint, TestPoint:TestPoint_Pad_D1.0mm
- added C7: 10u, Capacitor_SMD:C_0805_2012Metric_Pad1.15x1.40mm_HandSolder, F.Cu at (135.0, 93.5)
- added C8: 0.1u, Capacitor_SMD:C_0603_1608Metric_Pad1.05x0.95mm_HandSolder, F.Cu at (138.5, 93.5)
- added D1: LED, LED_SMD:LED_0603_1608Metric_Pad1.05x0.95mm_HandSolder, F.Cu at (119.0, 82.4)
- added D10: LED, LED_SMD:LED_0603_1608Metric_Pad1.05x0.95mm_HandSolder, F.Cu at (114.8, 95.9)
- added D2: LED, LED_SMD:LED_0603_1608Metric_Pad1.05x0.95mm_HandSolder, F.Cu at (108.4, 76.5)
- added D3: LED, LED_SMD:LED_0603_1608Metric_Pad1.05x0.95mm_HandSolder, F.Cu at (119.0, 80.6)
- added D4: LED, LED_SMD:LED_0603_1608Metric_Pad1.05x0.95mm_HandSolder, F.Cu at (119.0, 78.8)
- added D5: LED, LED_SMD:LED_0603_1608Metric_Pad1.05x0.95mm_HandSolder, F.Cu at (119.0, 86.2)
- added D6: LED, LED_SMD:LED_0603_1608Metric_Pad1.05x0.95mm_HandSolder, F.Cu at (119.0, 84.4)
- added D7: LED, LED_SMD:LED_0603_1608Metric_Pad1.05x0.95mm_HandSolder, F.Cu at (119.0, 77.0)
- added D8: LED, LED_SMD:LED_0603_1608Metric_Pad1.05x0.95mm_HandSolder, F.Cu at (85.1, 86.0)
- added D9: LED, LED_SMD:LED_0603_1608Metric_Pad1.05x0.95mm_HandSolder, F.Cu at (112.2, 95.9)
- added J7: Conn_01x03, Connector_PinHeader_2.54mm:PinHeader_1x03_P2.54mm_Vertical, F.Cu at (81.0, 90.5)
- added R10: 330, Resistor_SMD:R_0603_1608Metric_Pad1.05x0.95mm_HandSolder, F.Cu at (123.0, 84.4)
- added R11: 330, Resistor_SMD:R_0603_1608Metric_Pad1.05x0.95mm_HandSolder, F.Cu at (123.0, 77.0)
- added R12: 330, Resistor_SMD:R_0603_1608Metric_Pad1.05x0.95mm_HandSolder, F.Cu at (85.1, 83.5)
- added R16: 330, Resistor_SMD:R_0603_1608Metric_Pad1.05x0.95mm_HandSolder, F.Cu at (112.2, 91.6)
- added R17: 330, Resistor_SMD:R_0603_1608Metric_Pad1.05x0.95mm_HandSolder, F.Cu at (114.8, 91.7)
- added R5: 330, Resistor_SMD:R_0603_1608Metric_Pad1.05x0.95mm_HandSolder, F.Cu at (123.0, 82.4)
- added R6: 330, Resistor_SMD:R_0603_1608Metric_Pad1.05x0.95mm_HandSolder, F.Cu at (108.4, 74.5)
- added R7: 330, Resistor_SMD:R_0603_1608Metric_Pad1.05x0.95mm_HandSolder, F.Cu at (123.0, 80.6)
- added R8: 330, Resistor_SMD:R_0603_1608Metric_Pad1.05x0.95mm_HandSolder, F.Cu at (123.1, 78.8)
- added R9: 330, Resistor_SMD:R_0603_1608Metric_Pad1.05x0.95mm_HandSolder, F.Cu at (123.0, 86.2)
- J3: value Conn_02x20_Odd_Even -> Conn_Coaxial; footprint Connector_Molex:Molex_SlimStack_501920-4001_2x20_P0.50mm_Vertical -> Connector_Coaxial:SMA_Amphenol_132289_EdgeMount
- J4: value CONN_01X02 -> Conn_01x03; footprint Connector_PinHeader_2.54mm:PinHeader_1x02_P2.54mm_Vertical -> Connector_PinHeader_2.54mm:PinHeader_1x03_P2.54mm_Vertical
- J6: value CONN_01X02 -> Conn_01x06; footprint Connector_PinHeader_2.54mm:PinHeader_1x02_P2.54mm_Vertical -> Connector_PinHeader_2.54mm:PinHeader_1x06_P2.54mm_Vertical
- R13: value R -> 10K
- U3: value TS5A23159 -> RFM95W-915S2; footprint Package_SO:VSSOP-10_3x3mm_P0.5mm -> RF_Module:HOPERF_RFM9XW_SMD
- moved J6 54.1 mm to (127.5, 69.5), turned to 90 degrees
- moved TP3 46.5 mm to (81.0, 86.0), turned to 0 degrees
- moved TP5 42.9 mm to (81.0, 81.5)
- moved C3 35.5 mm to (85.0, 80.5)
- moved C4 35.0 mm to (85.0, 78.5)
- moved R14 34.7 mm to (84.6, 76.5)
- moved R15 34.6 mm to (88.4, 76.5)
- moved U2 34.5 mm to (83.5, 72.5)
- moved C2 33.5 mm to (81.1, 76.5)
- moved C1 32.6 mm to (85.0, 69.0)
- moved TP1 32.6 mm to (105.0, 91.4)
- moved R13 32.1 mm to (81.0, 69.0)
- moved U3 31.4 mm to (134.0, 81.5), turned to 270 degrees
- moved TP2 26.8 mm to (107.2, 91.4)
- moved C6 18.1 mm to (96.8, 75.0), turned to 180 degrees
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Connections:
- J2 pad 11: /GPS_RESETn -> /HAT_PG
- J2 pad 13: /GPS_WAKE -> /GPS_PPS
- J2 pad 15: /UART_MUX -> /GPS_RESETn
- J2 pad 17: (no net) -> /GPS_WAKE
- J2 pad 18: (no net) -> /PI_LED_2
- J2 pad 19: /HAT_PG -> /PI_LED_1
- J2 pad 21: /HAT_PWR_EN -> (no net)
- J2 pad 24: (no net) -> /SS
- J2 pad 29: /WAKEUP -> (no net)
- J2 pad 3: /GPS_SDA -> /I2C_SDA
- J2 pad 31: (no net) -> /RFM_RESET
- J2 pad 32: /BL_ENABLE -> (no net)
- J2 pad 33: /GPIO0 -> (no net)
- J2 pad 35: (no net) -> /MISO
- J2 pad 36: /GPIO1 -> (no net)
- J2 pad 37: /RESET_N -> (no net)
- J2 pad 38: (no net) -> /MOSI
- J2 pad 40: (no net) -> /SCLK
- J2 pad 5: /GPS_SCL -> /I2C_SCL
- J2 pad 7: /GPS_PPS -> /HAT_PWR_EN
- J3 pad 1: +3V3 -> Net-(J3-Pad1)
- J3 pad 2: /RESET_N -> GND
- J4 pad 1: /UART_RXD -> GND
- J6 pad 1: /GPS_SDA -> GND
- J6 pad 2: /GPS_SCL -> /RFM_RESET
- TP1 pad 1: /GPIO1 -> Net-(TP1-Pad1)
- TP2 pad 1: /BL_ENABLE -> Net-(TP2-Pad1)
- TP3 pad 1: /GPIO0 -> GND
- U3 pad 1: /UART_MUX -> GND
- U3 pad 10: /UART_RXD -> GND
- U3 pad 2: /GRIM_RXD -> /MISO
- U3 pad 3: GND -> /MOSI
- U3 pad 4: /GRIM_TXD -> /SCLK
- U3 pad 5: /UART_MUX -> /SS
- U3 pad 6: /UART_TXD -> /RFM_RESET
- U3 pad 7: /GPS_TXD -> Net-(R11-Pad1)
- U3 pad 8: +3V3 -> GND
- U3 pad 9: /GPS_RXD -> Net-(J3-Pad1)
- U5 pad 16: /GPS_SDA -> Net-(TP1-Pad1)
- U5 pad 17: /GPS_SCL -> Net-(TP2-Pad1)
- U5 pad 2: /GPS_TXD -> /UART_TXD
- U5 pad 3: /GPS_RXD -> /UART_RXD
Routing:
- net /WAKEUP: track 81.6 -> 0.00 mm, vias 3 -> 0
- net /GPIO0: track 80.2 -> 0.00 mm, vias 3 -> 0
- net /BL_ENABLE: track 71.1 -> 0.00 mm, vias 1 -> 0
- net /GPIO1: track 68.6 -> 0.00 mm, vias 1 -> 0
- net /GPS_SCL: track 60.7 -> 0.00 mm, vias 1 -> 0
- net /GPS_SDA: track 58.6 -> 0.00 mm, vias 1 -> 0
- net /GRIM_TXD: track 47.6 -> 0.00 mm
- net /GRIM_RXD: track 47.6 -> 0.00 mm, vias 2 -> 0
- net +3V3: track 58.5 -> 98.9 mm, vias 6 -> 5
- net /RESET_N: track 32.0 -> 0.00 mm
- net /PI_LED_2: track 0.00 -> 31.9 mm, vias 0 -> 1
- net /I2C_SDA: track 0.00 -> 28.7 mm, vias 0 -> 2
- net /GPS_TXD: track 28.5 -> 0.00 mm, vias 2 -> 0
- net /SS: track 0.00 -> 27.5 mm
- net /I2C_SCL: track 0.00 -> 27.4 mm, vias 0 -> 2
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- removed copper zone on B.Cu, net +3V3
- removed copper zone on F.Cu, net +3V3
- removed copper zone on B.Cu, net /P5V_HAT
Other:
- board size 65 x 56 mm -> 65 x 38.2 mm
- board text added: "."
- board text added: "GND SDA SCL"
- board text added: "J6: GND RESET SS MISO MOSI SCLK"
- board text added: "PiRFHat-GPS Rev B Nick Butts Copyright 2019"
- board text added: "RXD TXD GND"
- board text removed: "3.3V"
- board text removed: "BL_ENABLE"
- board text removed: "GPIO0"
- board text removed: "GPIO1"
- board text removed: "PiRFHat Rev A"
- board text removed: "PiRFHat-GPS Rev A Nick Butts Copyright 2019"
- board text removed: "RXD"
- board text removed: "SCL"
- board text removed: "SDA"
- board text removed: "TXD"
- board text removed: "WAKEUP"
